File: hardware/USB_condom.kicad_pcb (KiCad board)
At the start: 2 copper layers, 32.5 x 16.6 mm, 25 parts, among them J1 USB_A, J2 USB_A, U1 TPS2514A, U2 TPD2E001, U3 TPS2561

Commit message: update labels
Parts:
- removed kibuzzard-644073E0 (x2): G***, kibuzzard-644073E0
- removed kibuzzard-64407430 (x2): G***, kibuzzard-64407430
- added kibuzzard-65CAA4BB: G***, kibuzzard-65CAA4BB, F.Cu at (154.7, 97.0)
- added kibuzzard-65CAA4FF: G***, kibuzzard-65CAA4FF, B.Cu at (131.8, 93.6)
- added kibuzzard-65CAA527: G***, kibuzzard-65CAA527, B.Cu at (133.6, 93.5)
- added kibuzzard-65CAA533: G***, kibuzzard-65CAA533, F.Cu at (154.8, 98.9)

Commit message: Move_Components
Parts:
- moved C6 2.55 mm to (143.7, 93.0), turned to 0 degrees
- moved D1 0.86 mm to (143.8, 89.9)
- moved R7 0.84 mm to (142.7, 89.9)
- moved R5 0.63 mm to (143.3, 95.0)
- moved R6 0.62 mm to (141.1, 89.7)
- moved C3 0.49 mm to (140.3, 97.5)
- moved C5 0.40 mm to (137.2, 92.3)
- moved C2 0.39 mm to (141.1, 90.9)
- moved C4 0.05 mm to (138.1, 97.5)
Routing:
- net GND: track 18.9 -> 21.8 mm
- net VBUS: track 21.8 -> 22.6 mm
- net +5V: track 40.1 -> 39.4 mm
- net Net-(U3-ILM): track 1.26 -> 1.83 mm
