File: hardware/pawprotector.kicad_sch (KiCad schematic)
At the start: 19 parts, among them J1 USB_A, J2 USB_A, U1 TPS2514A, U2 TPD2E001, U3 TPS2561

Commit message: feat(Hw):Bom_Updated
Parts:
- C2: LCSC# C576742 -> C16772
- D1: LCSC# C965790 -> C397045
- R5: LCSC# C100292 -> C93942
- R7: LCSC# C2935237 -> C106235
- U3: LCSC# (none) -> C140303
