File: hardware/pawprotector.kicad_sch (KiCad schematic)
At the start: 15 parts, among them U1 TPS259480AYWPR, U2 TVS2200DRVR(ES), U3 TVS2200DRVR(ES), U4 TYPE-C-31-G-10, U5 KH-TYPE-C-16P

Commit message: Revision #2
Parts:
- removed U4: TYPE-C-31-G-10, USB-C_Male:USB-C-SMD_TYPE-C-31-G-10, symbol TYPE-C-31-G-10:TYPE-C-31-G-10
- removed U5: KH-TYPE-C-16P, USB-C-FEMALE:USB-C-SMD_KH-TYPE-C-16P, symbol KH-TYPE-C-16P:KH-TYPE-C-16P
- added D2: ON, LED_SMD:LED_0402_1005Metric, symbol Device:LED
- added J1: USB_C_Receptacle, symbol Connector:USB_C_Receptacle
- added P1: USB_C_Plug, symbol Connector:USB_C_Plug
- added R8: 500, Resistor_SMD:R_0402_1005Metric, symbol Device:R
- C3: value 2.7nF -> 12nF
- C5: value 1uF -> 4.7uF
- R7: value 1K -> 500
Connections:
- net +5V: now also P1.A4 (VBUS), P1.A9 (VBUS), P1.B4 (VBUS), P1.B9 (VBUS)
- net CC1: now also U3.4 (VDD/IO), U3.5 (VDD/IO), U3.6 (VDD/IO), J1.A5 (CC1), P1.A5 (CC); no longer U2.4 (VDD/IO), U2.5 (VDD/IO), U2.6 (VDD/IO)
- net CC2: now also J1.B5 (CC2); no longer U3.4 (VDD/IO), U3.5 (VDD/IO), U3.6 (VDD/IO)
- net GND: now also J1.A1 (GND), J1.A12 (GND), J1.B1 (GND), J1.B12 (GND), J1.SH (SHIELD), P1.A1 (GND), P1.A12 (GND), P1.B1 (GND), P1.B12 (GND), P1.SH (SHIELD), R8.2
- net VBUS: now also U2.4 (VDD/IO), U2.5 (VDD/IO), U2.6 (VDD/IO), J1.A4 (VBUS), J1.A9 (VBUS), J1.B4 (VBUS), J1.B9 (VBUS)
- net FLT#: now reaches U1.4 (FLT#)
- net FLT#: now also D2.2 (A)
- new net: D2.1 (K), R8.1
- no-connect marks 14 -> 27
Other:
- moved on the sheet: C3, C4, R2, R3, R4

Commit message: Revision #2
Connections:
- net CC2: now also P1.B5 (VCONN)
Changed lines of the file:
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@@
 	(text "Diodes TVS\n"
 		(exclude_from_sim no)
-		(at 149.606 91.186 0)
+		(at 151.892 91.694 0)
 		(effects
 			(font
@@
 		)
 		(stroke
+			(width 0)
+			(type default)
+		)
+	)
+	(wire
+		(pts
+			(xy 46.99 39.37) (xy 53.34 39.37)
+		)
+		(stroke

Commit message: Revision #3
Parts:
- removed D2: ON, LED_SMD:LED_0402_1005Metric, symbol Device:LED
- removed R8: 500, Resistor_SMD:R_0402_1005Metric, symbol Device:R
- removed U3: TVS2200DRVR(ES), TVS2200:DFN-6_L2.0-W2.0-P0.65-BL-EP1.6, symbol TVS2200DRVR(ES):TVS2200DRVR(ES)
- added U3: ESD752DBZR, footprint:SOT-23-3_L2.9-W1.3-P1.90-LS2.4-BR, symbol ESD752DBZR:ESD752DBZR
- D1: LCSC# C397045 -> C25503345
- R7: value 500 -> 1k
Connections:
- net CC1: now also U3.1 (IO)
- net CC2: now also U3.2 (IO)
- net GND: now also U3.3 (GND)
- net FLT#: no longer names the net of U1.4 (FLT#)
- no-connect marks 27 -> 28
Other:
- moved on the sheet: C4

Commit message: Ruteo PCB
Parts:
- J1: footprint (none) -> USB-C-FEMALE:USB-C-SMD_KH-TYPE-C-16P
- P1: footprint (none) -> USB-C_Male:USB-C-SMD_TYPE-C-31-G-10
- U2: footprint TVS2200:DFN-6_L2.0-W2.0-P0.65-BL-EP1.6 -> TVS2200DRVR:DFN-6_L2.0-W2.0-P0.65-BL-EP1.6
- U3: footprint footprint:SOT-23-3_L2.9-W1.3-P1.90-LS2.4-BR -> ESD752DBZR:SOT-23-3_L2.9-W1.3-P1.90-LS2.4-BR
- renumbered C4 to C1, C3 to C2, C5 to C3, C2 to C4, R2 to R1, R3 to R2, R4 to R3, R1 to R4, R7 to R5
Connections:
- net CC1: now also U3.2 (IO); no longer U3.1 (IO)
- net CC2: now also U3.1 (IO); no longer U3.2 (IO)
Changed lines of the file:
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@@
 		)
 	)
-	(label "CC2"
+	(label "CC1"
 		(at 137.16 133.35 0)
 		(effects
@@
 		)
 	)
-	(label "CC1"
+	(label "CC2"
 		(at 137.16 130.81 0)
 		(effects
@@
 		(dnp no)
 		(fields_autoplaced yes)
-		(property "Reference" "#PWR08"
+		(property "Reference" "#PWR015"
 			(at 168.91 67.31 0)
 			(hide yes)
@@
 			(project "pawprotector"
 				(path "/0d5adc36-ef78-4419-baea-66b821882972"
-					(reference "#PWR08")
+					(reference "#PWR015")
 					(unit 1)
 				)
@@
 		(dnp no)
 		(fields_autoplaced yes)
-		(property "Reference" "#PWR05"
+		(property "Reference" "#PWR04"
 			(at 172.72 35.56 0)
 			(hide yes)
@@
 			(project "pawprotector"
 				(path "/0d5adc36-ef78-4419-baea-66b821882972"
-					(reference "#PWR05")
+					(reference "#PWR04")
 					(unit 1)
 				)
@@
 		(dnp no)
 		(fields_autoplaced yes)
-		(property "Reference" "#PWR022"
+		(property "Reference" "#PWR08"
 			(at 196.85 40.132 0)
 			(hide yes)
@@
 			(project "pawprotector"
 				(path "/0d5adc36-ef78-4419-baea-66b821882972"
-					(reference "#PWR022")
+					(reference "#PWR08")
 					(unit 1)
 				)
@@
 		(dnp no)
 		(fields_autoplaced yes)
-		(property "Reference" "#PWR04"
+		(property "Reference" "#PWR013"
 			(at 173.99 59.69 0)
 			(hide yes)
@@
 			(project "pawprotector"
 				(path "/0d5adc36-ef78-4419-baea-66b821882972"
-					(reference "#PWR04")
+					(reference "#PWR013")
 					(unit 1)
 				)
@@
 		(dnp no)
 		(fields_autoplaced yes)
-		(property "Reference" "R2"
+		(property "Reference" "R1"
 			(at 120.65 31.7499 0)
 			(show_name no)
@@
 			(project "pawprotector"
 				(path "/0d5adc36-ef78-4419-baea-66b821882972"
-					(reference "R2")
+					(reference "R1")
 					(unit 1)
 				)
@@
 		(dnp no)
 		(fields_autoplaced yes)
-		(property "Reference" "C4"
+		(property "Reference" "C1"
 			(at 92.71 40.6399 0)
 			(show_name no)
@@
 			(project "pawprotector"
 				(path "/0d5adc36-ef78-4419-baea-66b821882972"
-					(reference "C4")
+					(reference "C1")
 					(unit 1)
 				)
@@
 		(dnp no)
 		(fields_autoplaced yes)
-		(property "Reference" "#PWR037"
+		(property "Reference" "#PWR017"
 			(at 248.92 107.95 0)
 			(hide yes)
@@
 			(project "pawprotector"
 				(path "/0d5adc36-ef78-4419-baea-66b821882972"
-					(reference "#PWR037")
+					(reference "#PWR017")
 					(unit 1)
 				)
@@
 		(dnp no)
 		(fields_autoplaced yes)
-		(property "Reference" "#PWR012"
+		(property "Reference" "#PWR03"
 			(at 270.51 33.02 0)
 			(hide yes)
@@
 			(project "pawprotector"
 				(path "/0d5adc36-ef78-4419-baea-66b821882972"
-					(reference "#PWR012")
+					(reference "#PWR03")
 					(unit 1)
 				)
@@
 		(dnp no)
 		(fields_autoplaced yes)
-		(property "Reference" "#PWR07"
+		(property "Reference" "#PWR02"
 			(at 53.34 33.02 0)
 			(hide yes)
@@
 			(project "pawprotector"
 				(path "/0d5adc36-ef78-4419-baea-66b821882972"
-					(reference "#PWR07")
+					(reference "#PWR02")
 					(unit 1)
 				)
@@
 		(dnp no)
 		(fields_autoplaced yes)
-		(property "Reference" "#PWR025"
+		(property "Reference" "#PWR07"
 			(at 88.9 40.132 0)
 			(hide yes)
@@
 			(project "pawprotector"
 				(path "/0d5adc36-ef78-4419-baea-66b821882972"
-					(reference "#PWR025")
+					(reference "#PWR07")
 					(unit 1)
 				)
@@
 		(dnp no)
 		(fields_autoplaced yes)
-		(property "Reference" "#PWR024"
+		(property "Reference" "#PWR010"
 			(at 88.9 53.975 0)
 			(hide yes)
@@
 			(project "pawprotector"
 				(path "/0d5adc36-ef78-4419-baea-66b821882972"
-					(reference "#PWR024")
+					(reference "#PWR010")
 					(unit 1)
 				)
@@
 		(dnp no)
 		(fields_autoplaced yes)
-		(property "Reference" "#PWR039"
+		(property "Reference" "#PWR016"
 			(at 31.75 107.95 0)
 			(hide yes)
@@
 			(project "pawprotector"
 				(path "/0d5adc36-ef78-4419-baea-66b821882972"
-					(reference "#PWR039")
+					(reference "#PWR016")
 					(unit 1)
 				)
@@
 		(dnp no)
 		(fields_autoplaced yes)
-		(property "Reference" "#PWR010"
+		(property "Reference" "#PWR01"
 			(at 118.11 31.75 0)
 			(hide yes)
@@
 			(project "pawprotector"
 				(path "/0d5adc36-ef78-4419-baea-66b821882972"
-					(reference "#PWR010")
+					(reference "#PWR01")
 					(unit 1)
 				)
@@
 		(in_pos_files yes)
 		(dnp no)
-		(property "Reference" "C2"
+		(property "Reference" "C4"
 			(at 162.56 53.34 0)
 			(show_name no)
@@
 			(project "pawprotector"
 				(path "/0d5adc36-ef78-4419-baea-66b821882972"
-					(reference "C2")
+					(reference "C4")
 					(unit 1)
 				)
@@
 		(in_pos_files yes)
 		(dnp no)
-		(property "Reference" "C5"
+		(property "Reference" "C3"
 			(at 190.5 40.64 0)
 			(show_name no)
@@
 			(project "pawprotector"
 				(path "/0d5adc36-ef78-4419-baea-66b821882972"
-					(reference "C5")
+					(reference "C3")
 					(unit 1)
 				)
@@
 		(dnp no)
 		(fields_autoplaced yes)
-		(property "Reference" "#PWR031"
+		(property "Reference" "#PWR05"
 			(at 214.63 37.973 0)
 			(hide yes)
@@
 			(project "pawprotector"
 				(path "/0d5adc36-ef78-4419-baea-66b821882972"
-					(reference "#PWR031")
+					(reference "#PWR05")
 					(unit 1)
 				)
@@
 		(dnp no)
 		(fields_autoplaced yes)
-		(property "Reference" "C3"
+		(property "Reference" "C2"
 			(at 106.68 40.6399 0)
 			(show_name no)
@@
 			(project "pawprotector"
 				(path "/0d5adc36-ef78-4419-baea-66b821882972"
-					(reference "C3")
+					(reference "C2")
 					(unit 1)
 				)
@@
 		(dnp no)
 		(fields_autoplaced yes)
-		(property "Reference" "#PWR023"
+		(property "Reference" "#PWR09"
 			(at 196.85 53.848 0)
 			(hide yes)
@@
 			(project "pawprotector"
 				(path "/0d5adc36-ef78-4419-baea-66b821882972"
-					(reference "#PWR023")
+					(reference "#PWR09")
 					(unit 1)
 				)
@@
 		(dnp no)
 		(fields_autoplaced yes)
-		(property "Reference" "#PWR028"
+		(property "Reference" "#PWR012"
 			(at 214.63 59.182 0)
 			(hide yes)
@@
 			(project "pawprotector"
 				(path "/0d5adc36-ef78-4419-baea-66b821882972"
-					(reference "#PWR028")
+					(reference "#PWR012")
 					(unit 1)
 				)
@@
 		(dnp no)
 		(fields_autoplaced yes)
-		(property "Reference" "#PWR03"
+		(property "Reference" "#PWR019"
 			(at 162.56 139.7 0)
 			(hide yes)
@@
 			(project "pawprotector"
 				(path "/0d5adc36-ef78-4419-baea-66b821882972"
-					(reference "#PWR03")
+					(reference "#PWR019")
 					(unit 1)
 				)
@@
 		(in_pos_files yes)
 		(dnp no)
-		(property "Reference" "R7"
+		(property "Reference" "R5"
 			(at 210.947 46.355 0)
 			(show_name no)
@@
 			(project "pawprotector"
 				(path "/0d5adc36-ef78-4419-baea-66b821882972"
-					(reference "R7")
+					(reference "R5")
 					(unit 1)
 				)
@@
 		(dnp no)
 		(fields_autoplaced yes)
-		(property "Reference" "R4"
+		(property "Reference" "R3"
 			(at 120.65 52.0699 0)
 			(show_name no)
@@
 			(project "pawprotector"
 				(path "/0d5adc36-ef78-4419-baea-66b821882972"
-					(reference "R4")
+					(reference "R3")
 					(unit 1)
 				)
@@
 		(dnp no)
 		(fields_autoplaced yes)
-		(property "Reference" "#PWR09"
+		(property "Reference" "#PWR014"
 			(at 118.11 66.04 0)
 			(hide yes)
@@
 			(project "pawprotector"
 				(path "/0d5adc36-ef78-4419-baea-66b821882972"
-					(reference "#PWR09")
+					(reference "#PWR014")
 					(unit 1)
 				)
@@
 			)
 		)
-		(property "Footprint" "TVS2200:DFN-6_L2.0-W2.0-P0.65-BL-EP1.6"
+		(property "Footprint" "TVS2200DRVR:DFN-6_L2.0-W2.0-P0.65-BL-EP1.6"
 			(at 151.13 118.11 0)
 			(hide yes)
@@
 		(dnp no)
 		(fields_autoplaced yes)
-		(property "Reference" "R3"
+		(property "Reference" "R2"
 			(at 120.65 41.9099 0)
 			(show_name no)
@@
 			(project "pawprotector"
 				(path "/0d5adc36-ef78-4419-baea-66b821882972"
-					(reference "R3")
+					(reference "R2")
 					(unit 1)
 				)
@@
 			)
 		)
-		(property "Footprint" "footprint:SOT-23-3_L2.9-W1.3-P1.90-LS2.4-BR"
+		(property "Footprint" "ESD752DBZR:SOT-23-3_L2.9-W1.3-P1.90-LS2.4-BR"
 			(at 151.13 142.24 0)
 			(hide yes)
@@
 		(dnp no)
 		(fields_autoplaced yes)
-		(property "Reference" "#PWR01"
+		(property "Reference" "#PWR018"
 			(at 134.62 119.38 0)
 			(hide yes)
@@
 			(project "pawprotector"
 				(path "/0d5adc36-ef78-4419-baea-66b821882972"
-					(reference "#PWR01")
+					(reference "#PWR018")
 					(unit 1)
 				)
@@
 			)
 		)
-		(property "Footprint" ""
+		(property "Footprint" "USB-C-FEMALE:USB-C-SMD_KH-TYPE-C-16P"
 			(at 252.73 57.15 0)
 			(hide yes)
@@
 			)
 		)
-		(property "Footprint" ""
+		(property "Footprint" "USB-C_Male:USB-C-SMD_TYPE-C-31-G-10"
 			(at 35.56 57.15 0)
 			(hide yes)
@@
 		(dnp no)
 		(fields_autoplaced yes)
-		(property "Reference" "R1"
+		(property "Reference" "R4"
 			(at 176.53 45.7199 0)
 			(show_name no)
@@
 			(project "pawprotector"
 				(path "/0d5adc36-ef78-4419-baea-66b821882972"
-					(reference "R1")
+					(reference "R4")
 					(unit 1)
 				)

Commit message: feat(Hw): Bom_Updated
Parts:
- C2: LCSC# C106251 -> C880620
- C3: footprint Capacitor_SMD:C_0603_1608Metric -> Capacitor_SMD:C_0805_2012Metric; LCSC# C5199872 -> C513770
- J1: LCSC# (none) -> C709357
- P1: LCSC# (none) -> C5370430
- U3: LCSC# (none) -> C20345397
Changed lines of the file:
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@@
 			)
 		)
-		(property "Footprint" "Capacitor_SMD:C_0603_1608Metric"
+		(property "Footprint" "Capacitor_SMD:C_0805_2012Metric"
 			(at 197.8152 45.72 0)
 			(hide yes)
@@
 			)
 		)
-		(property "LCSC#" "C5199872"
+		(property "LCSC#" "C513770"
 			(at 196.85 41.91 0)
 			(hide yes)
@@
 			)
 		)
-		(property "LCSC#" "C106251"
+		(property "LCSC#" "C880620"
 			(at 102.87 41.91 0)
 			(hide yes)
@@
 			)
 		)
+		(property "LCSC#" "C20345397"
+			(at 151.13 132.08 0)
+			(hide yes)
+			(show_name no)
+			(do_not_autoplace no)
+			(effects
+				(font
+					(size 1.27 1.27)
+				)
+			)
+		)
 		(pin "1"
 		)
@@
 			)
 		)
+		(property "LCSC#" "C709357"
+			(at 248.92 57.15 0)
+			(hide yes)
+			(show_name no)
+			(do_not_autoplace no)
+			(effects
+				(font
+					(size 1.27 1.27)
+				)
+			)
+		)
 		(pin "A7"
 		)
@@
 			(at 31.75 57.15 0)
 			(hide yes)
+			(show_name no)
+			(do_not_autoplace no)
+			(effects
+				(font
+					(size 1.27 1.27)
+				)
+			)
+		)
+		(property "LCSC#" "C5370430"
+			(at 31.75 57.15 0)
+			(hide yes)
